File: imu.kicad_sch (KiCad schematic)
At the start: 5 parts, among them U3 LSM6DSV320XTR

Commit message: clean up schematics and start pcb
Parts:
- C10, C9: footprint (none) -> Capacitor_SMD:C_0805_2012Metric_Pad1.18x1.45mm_HandSolder
- R13, R14: footprint (none) -> Resistor_SMD:R_0805_2012Metric_Pad1.20x1.40mm_HandSolder
- U3: footprint LGA-14L_2p5X3X0p83_STM -> footprints:LGA-14L_2p5X3X0p83_STM
Changed lines of the file:
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@@
 			)
 		)
-		(property "Footprint" "LGA-14L_2p5X3X0p83_STM"
+		(property "Footprint" "footprints:LGA-14L_2p5X3X0p83_STM"
 			(at 45.72 40.64 0)
 			(hide yes)
@@
 			)
 		)
-		(property "Footprint" ""
+		(property "Footprint" "Capacitor_SMD:C_0805_2012Metric_Pad1.18x1.45mm_HandSolder"
 			(at 108.9152 63.5 0)
 			(hide yes)
@@
 			)
 		)
-		(property "Footprint" ""
+		(property "Footprint" "Capacitor_SMD:C_0805_2012Metric_Pad1.18x1.45mm_HandSolder"
 			(at 33.9852 58.42 0)
 			(hide yes)
@@
 			)
 		)
-		(property "Footprint" ""
+		(property "Footprint" "Resistor_SMD:R_0805_2012Metric_Pad1.20x1.40mm_HandSolder"
 			(at 40.132 36.83 90)
 			(hide yes)
@@
 			)
 		)
-		(property "Footprint" ""
+		(property "Footprint" "Resistor_SMD:R_0805_2012Metric_Pad1.20x1.40mm_HandSolder"
 			(at 55.372 82.55 90)
 			(hide yes)
