File: subsheets/power.kicad_sch (KiCad schematic)
At the start: 30 parts, among them J1 Battery Connector, J10 VBAT_ESC_C, J11 VBAT_ESC_E, J12 VBAT_ESC_F, J13 VBAT_ESC_G, J14 VBAT_ESC_D, J15 VBAT_ESC_H, J8 VBAT_ESC_A, J9 VBAT_ESC_B, SW1 FingerTech Switch, U2 TPS563200

Commit message: Thicken power traces and some cleanup
Connections:
- net VBUS: now also SW1.2 (B); no longer SW1.1 (A)
- net at J1.1 (Pin_1): now also SW1.1 (A); no longer SW1.2 (B)
Changed lines of the file:
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@@
 		(color 0 0 0 0)
+	)
+	(bus_entry
+		(at 80.01 46.99)
+		(size 2.54 2.54)
+		(stroke
+			(width 0)
+			(type default)
+		)
 	)
 	(wire
@@
 		(lib_id "Switch:SW_SPST")
 		(at 62.23 33.02 0)
+		(mirror y)
 		(unit 1)
 		(body_style 1)
@@
 		(dnp no)
 		(property "Reference" "SW1"
-			(at 62.23 26.67 0)
-			(show_name no)
-			(do_not_autoplace no)
+			(at 72.39 26.67 0)
+			(show_name no)
+			(do_not_autoplace no)
